File: circuit/atarimovie.brd (EAGLE design)
At the start: 72.4 x 82.5 mm, 11 parts, among them X1 22-23-2051

Commit message: Using PIC18F47K42 not PIC18F45K42
Parts:
- U$1: value PIC18F45K42 -> PIC18F47K42
Changed lines of the file:
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@@
 </autorouter>
 <elements>
-<element name="U$1" library="atari" package="DIP40" value="PIC18F45K42" x="44.577" y="71.12" rot="R90.1"/>
+<element name="U$1" library="atari" package="DIP40" value="PIC18F47K42" x="44.577" y="71.12" rot="R90.1"/>
 <element name="U$2" library="atari" package="DIP48" value="7130LA35PDG" x="40.64" y="50.8" rot="R90"/>
 <element name="JP1" library="sparkfun" package="USD_SHIFTER" value="" x="38.1" y="29.21" smashed="yes" rot="R270">
